File: bleached ++ kicad files/bleachedplusplus.sch (KiCad schematic (older format))
At the start: 10 parts, among them U1 Teensy-LC_minimal

Commit message: Add files via upload
fixed potentiometer rotation
Connections:
- net +3V3: now also RV1.3, RV2.3, RV3.3, RV4.3, RV5.3, RV6.3, RV7.3, RV8.3, RV9.3; no longer RV1.1, RV2.1, RV3.1, RV4.1, RV5.1, RV6.1, RV7.1, RV8.1, RV9.1
- net GND: now also RV1.1, RV2.1, RV3.1, RV4.1, RV5.1, RV6.1, RV7.1, RV8.1, RV9.1; no longer RV1.3, RV2.3, RV3.3, RV4.3, RV5.3, RV6.3, RV7.3, RV8.3, RV9.3
Changed lines of the file:
@@
 F 3 "~" H 5000 2850 50  0001 C CNN
 	1    5000 2850
-	1    0    0    -1
+	1    0    0    1
 $EndComp
 $Comp
@@
 F 3 "~" H 6000 2850 50  0001 C CNN
 	1    6000 2850
-	1    0    0    -1
+	1    0    0    1
 $EndComp
 $Comp
@@
 F 3 "~" H 7000 2850 50  0001 C CNN
 	1    7000 2850
-	1    0    0    -1
+	1    0    0    1
 $EndComp
 $Comp
@@
 F 3 "~" H 8000 2850 50  0001 C CNN
 	1    8000 2850
-	1    0    0    -1
+	1    0    0    1
 $EndComp
 $Comp
@@
 F 3 "~" H 9000 2850 50  0001 C CNN
 	1    9000 2850
-	1    0    0    -1
+	1    0    0    1
 $EndComp
 $Comp
@@
 F 3 "~" H 5000 3910 50  0001 C CNN
 	1    5000 3910
-	1    0    0    -1
+	1    0    0    1
 $EndComp
 $Comp
@@
 F 3 "~" H 6000 3910 50  0001 C CNN
 	1    6000 3910
-	1    0    0    -1
+	1    0    0    1
 $EndComp
 $Comp
@@
 F 3 "~" H 7000 3910 50  0001 C CNN
 	1    7000 3910
-	1    0    0    -1
+	1    0    0    1
 $EndComp
 $Comp
@@
 F 3 "~" H 8000 3910 50  0001 C CNN
 	1    8000 3910
-	1    0    0    -1
-$EndComp
-$Comp
+	1    0    0    1
+$EndComp
+$Comp

Commit message: Add files via upload
Parts:
- added H1, H2, H3, H4: MountingHole, MountingHole:MountingHole_2.7mm_M2.5_DIN965_Pad, symbol Mechanical:MountingHole
Changed lines of the file:
@@
 	1080 2940 1080 2950
 NoConn ~ 3760 3730
+$Comp
+L Mechanical:MountingHole H2
+U 1 1 6130E76A
+P 8760 5340
+F 0 "H2" H 8860 5386 50  0000 L CNN
+F 1 "MountingHole" H 8860 5295 50  0000 L CNN
+F 2 "MountingHole:MountingHole_2.7mm_M2.5_DIN965_Pad" H 8760 5340 50  0001 C CNN
+F 3 "~" H 8760 5340 50  0001 C CNN
+	1    8760 5340
+	1    0    0    -1
+$EndComp
+$Comp
+L Mechanical:MountingHole H1
+U 1 1 6130F911
+P 9660 5330
+F 0 "H1" H 9760 5376 50  0000 L CNN
+F 1 "MountingHole" H 9760 5285 50  0000 L CNN
+F 2 "MountingHole:MountingHole_2.7mm_M2.5_DIN965_Pad" H 9660 5330 50  0001 C CNN
+F 3 "~" H 9660 5330 50  0001 C CNN
+	1    9660 5330
+	1    0    0    -1
+$EndComp
+$Comp
+L Mechanical:MountingHole H3
+U 1 1 6130FB77
+P 8760 5630
+F 0 "H3" H 8860 5676 50  0000 L CNN
+F 1 "MountingHole" H 8860 5585 50  0000 L CNN
+F 2 "MountingHole:MountingHole_2.7mm_M2.5_DIN965_Pad" H 8760 5630 50  0001 C CNN
+F 3 "~" H 8760 5630 50  0001 C CNN
+	1    8760 5630
+	1    0    0    -1
+$EndComp
+$Comp
+L Mechanical:MountingHole H4
+U 1 1 6130FCD8
+P 9670 5650
+F 0 "H4" H 9770 5696 50  0000 L CNN
+F 1 "MountingHole" H 9770 5605 50  0000 L CNN
+F 2 "MountingHole:MountingHole_2.7mm_M2.5_DIN965_Pad" H 9670 5650 50  0001 C CNN
+F 3 "~" H 9670 5650 50  0001 C CNN
+	1    9670 5650
+	1    0    0    -1
+$EndComp
 $EndSCHEMATC
